File: Docs/Documents & Advanced/PCB/V3.3/einkPDA_keyboard/einkPDA_keyboard.kicad_sch (KiCad schematic)
At the start: 126 parts, among them J1 USB_C_Receptacle_USB2.0_16P, J2 Conn_01x12_Pin, J3 Conn_01x26_Pin, J4 Micro_SD_Card, J5 Conn_01x12_Pin, Q1 MMBT3904, SW36 YTS-C017-2B, SW4 SW_DIP_x02, U1 ESP32-S3-WROOM-1, U10 TS3USB30ERSWR, U2 USBLC6-2SC6, U3 TPS63001, U4 PCF8563T, U5 TCA8418RTWR, U6 C2764211, U7 TPS61040DBV, U9 MP2722GRH-0000-Z, Y1 Crystal_32.768kHz

Commit message: Update PCB
Parts:
- removed JP1: SolderJumper_2_Open, Jumper:SolderJumper-2_P1.3mm_Open_RoundedPad1.0x1.5mm, symbol Jumper:SolderJumper_2_Open
- removed R9: 10K, Resistor_SMD:R_0805_2012Metric, symbol 0805W8F1002T5E:0805W8F1002T5E
- added C18: 680pF, Capacitor_SMD:C_0805_2012Metric, symbol Device:C
- added C33: 0.1uF, Capacitor_SMD:C_0402_1005Metric, symbol Device:C
- added C4: 1uF, Capacitor_SMD:C_0603_1608Metric, symbol Device:C
- added C5: 47uF, Capacitor_SMD:C_0805_2012Metric, symbol Device:C
- added JP1, JP10: SolderJumper_2_Bridged, Jumper:SolderJumper-2_P1.3mm_Bridged_RoundedPad1.0x1.5mm, symbol Jumper:SolderJumper_2_Bridged
- added JP2, JP7, JP8, JP9: SolderJumper_2_Open, Jumper:SolderJumper-2_P1.3mm_Open_RoundedPad1.0x1.5mm, symbol Jumper:SolderJumper_2_Open
- added R19: 100K, Resistor_SMD:R_0603_1608Metric, symbol Device:R
- added R4: 1k, Resistor_SMD:R_0603_1608Metric, symbol Device:R
- added R5: 470R, Resistor_SMD:R_0805_2012Metric, symbol Device:R
- added R9: 10k, Resistor_SMD:R_0805_2012Metric, symbol Device:R
- added SW41: YTS-C017-2B, customparts:KEY-TH_3P-L4.5-W4.5-P3.0-EH, symbol CustomParts:YTS-C017-2B
- added U8: TPS22917DBV, Package_TO_SOT_SMD:SOT-23-6, symbol Power_Management:TPS22917DBV
- R10: value 20k -> 10k; footprint Resistor_SMD:R_0603_1608Metric -> Resistor_SMD:R_0805_2012Metric; LCSC Part # C4184 -> C17414
Connections:
- net +3.3V: now also R10.2, C18.1, C4.2, JP2.2 (B), JP7.2 (B), JP8.2 (B), JP9.2 (B), R9.1, U8.1 (VIN); no longer C10.2, C16.1, C17.1, C21.2, C22.2, C24.1, J2.12 (Pin_12), J3.21 (Pin_21), J3.22 (Pin_22), J4.4 (VDD), J5.1 (Pin_1), L1.1, U7.4 (EN), U7.5 (VIN)
- net CHRG: no longer R10.1
- net EN: now also C33.1, SW41.1
- net EX_D: now also U1.35 (IO42); no longer U1.6 (IO6)
- net EX_E: now also U1.25 (IO48); no longer U1.5 (IO5)
- net GND: now also C33.2, C4.1, C5.2, R19.2, R4.2, SW41.2, SW41.3 (GND), U8.2 (GND); no longer R10.2
- net SD_CLK: now also RN3.8 (R1.2); no longer JP3.1 (A)
- net SD_CS: now also JP1.1 (A)
- net at JP3.2 (B): now also R10.1; no longer RN3.8 (R1.2)
- net at J4.2 (DAT3/CD), RN3.7 (R2.2): now also JP1.2 (B)
- net SD_D2: now reaches J4.1 (DAT2)
- net SD_D2: now also JP3.1 (A), U1.6 (IO6)
- net SD_D1: now reaches J4.8 (DAT1)
- net SD_D1: now also U1.5 (IO5), JP10.1 (A)
- net LOAD: now reaches U1.31 (IO38)
- net LOAD: now also R19.1, U8.3 (ON)
- new net: JP10.2 (B), R9.2
- new net: R5.2, U8.5 (QOD)
- new net: C18.2, U8.4 (CT)
- new net V_LOADSWITCH: C10.2, C16.1, C17.1, C21.2, C22.2, C24.1, C5.1, J2.12 (Pin_12), J3.21 (Pin_21), J3.22 (Pin_22), J4.4 (VDD), J5.1 (Pin_1), JP2.1 (A), JP7.1 (A), JP8.1 (A), JP9.1 (A), L1.1, R4.1, R5.1, U7.4 (EN), U7.5 (VIN), U8.6 (VOUT)
- no-connect marks 11 -> 9
Other:
- note added: "Sleep & RST Button"
- note added: "Sleep Load Switch"
- note removed: "Plug Sensing"
- note removed: "Sleep Button"
- moved on the sheet: C19, C21, C22, C24, C6, C8, D5, FB2, J2, R14, R18, R3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
